Commit message: add inertia to the urdf

File: src/my_robot_description/urdf/common_properties.xacro (robot description, xacro)
@@ -7,3 +7,30 @@
         <color rgba="0.5 0.5 0.5 1" />
     </material>
+    <xacro:macro name="box_inertia" params="m l w h xyz rpy">
+        <inertial>
+            <origin xyz="${xyz}" rpy="${rpy}" />
+            <mass value="${m}" />
+            <inertia ixx="${(m/12) * h*h + l*l}" ixy="0" ixz="0"
+                     iyy="${(m/12) * (w*w + l*l)}" iyz="0"
+                     izz="${(m/12) * (w*w + h*h)}"/>
+        </inertial>
+    </xacro:macro>
+    <xacro:macro name="cylinder_inertia" params="m r h xyz rpy">
+        <inertial>
+            <origin xyz="${xyz}" rpy="${rpy}" />
+            <mass value="${m}" />
+            <inertia ixx="${m/12 * (3 * r*r+ h*h)}" ixy="0" ixz="0"
+                     iyy="${m/12 * (3 * r*r+ h*h)}" iyz="0"
+                     izz="${0.5 * m * r*r}" />
+        </inertial>
+    </xacro:macro>
+    <xacro:macro name="sphere_inertia" params="m r xyz rpy">
+        <inertial>
+            <origin xyz="${xyz}" rpy="${rpy}" />
+            <mass value="${m}" />
+            <inertia ixx="${2/5 * m * r*r}" ixy="0" ixz="0"
+                     iyy="${2/5 * m * r*r}" iyz="0"
+                     izz="${2/5 * m * r*r}" />
+        </inertial>
+    </xacro:macro>
 </robot>

File: src/my_robot_description/urdf/mobile_base.xacro (robot description, xacro)
@@ -16,4 +16,6 @@
             <material name="green" />
         </visual>
+        <xacro:box_inertia m="5.0" l="${base_length}" w="${base_width}" h="${base_height}"
+                            xyz="0 0 ${wheel_radius}" rpy="0 0 0" />
     </link>
     <joint name="base_base_foot_plane" type="fixed">
@@ -31,4 +33,5 @@
                 <material name="grey" />
             </visual>
+            <xacro:cylinder_inertia m="1.0" r="${wheel_radius}" h="${wheel_length}" xyz="0 0 0" rpy="${pi / 2.0} 0 0"/>
         </link>
     </xacro:macro>
@@ -55,4 +58,5 @@
             <material name="grey" />
         </visual>
+        <xacro:sphere_inertia m="0.5" r="${wheel_radius / 2}" xyz="0 0 0" rpy="0 0 0" />
     </link>
     <joint name="base_front_caster_wheel" type="fixed">

Commit message: fix the problem of incorrect inertia error

File: src/my_robot_description/urdf/common_properties.xacro (robot description, xacro)
@@ -11,7 +11,7 @@
             <origin xyz="${xyz}" rpy="${rpy}" />
             <mass value="${m}" />
-            <inertia ixx="${(m/12) * h*h + l*l}" ixy="0" ixz="0"
-                     iyy="${(m/12) * (w*w + l*l)}" iyz="0"
-                     izz="${(m/12) * (w*w + h*h)}"/>
+            <inertia ixx="${(m/12) * (h*h + l*l)}" ixy="0" ixz="0"
+                     iyy="${(m/12) * (w*w + h*h)}" iyz="0"
+                     izz="${(m/12) * (w*w + l*l)}"/>
         </inertial>
     </xacro:macro>
