Commit message: change front wheel size

File: src/my_robot_description/urdf/mobile_base.xacro (robot description, xacro)
@@ -50,5 +50,5 @@
         <visual>
             <geometry>
-                <sphere radius="${wheel_radius}"/>
+                <sphere radius="${wheel_radius / 2}"/>
             </geometry>
             <origin xyz="0 0 0" rpy="0 0 0" />

Commit message: add online URDF into the gazebo with service call, check my_robot xacro file error

File: src/my_robot_description/urdf/mobile_base.xacro (robot description, xacro)
@@ -16,4 +16,10 @@
             <material name="green" />
         </visual>
+        <collision>
+            <geometry>
+                <box size="${base_length} ${base_width} ${base_height}" />
+            </geometry>
+            <origin xyz="0 0 ${wheel_radius}" rpy="0 0 0" />
+        </collision>
         <xacro:box_inertia m="5.0" l="${base_length}" w="${base_width}" h="${base_height}"
                             xyz="0 0 ${wheel_radius}" rpy="0 0 0" />
@@ -33,4 +39,10 @@
                 <material name="grey" />
             </visual>
+            <collision>
+                <geometry>
+                    <cylinder radius="${wheel_radius}" length="${wheel_length}" />
+                </geometry>
+                <origin xyz="0 0 0" rpy="${pi / 2.0} 0 0" />
+            </collision>
             <xacro:cylinder_inertia m="1.0" r="${wheel_radius}" h="${wheel_length}" xyz="0 0 0" rpy="${pi / 2.0} 0 0"/>
         </link>
@@ -58,4 +70,10 @@
             <material name="grey" />
         </visual>
+        <collision>
+            <geometry>
+                <sphere radius="${wheel_radius / 2}"/>
+            </geometry>
+            <origin xyz="0 0 0" rpy="0 0 0" />
+        </collision>
         <xacro:sphere_inertia m="0.5" r="${wheel_radius / 2}" xyz="0 0 0" rpy="0 0 0" />
     </link>

Commit message: wrap earlier work

File: src/my_robot_description/urdf/mobile_base.xacro (robot description, xacro)
@@ -6,6 +6,5 @@
     <xacro:property name="wheel_radius" value="0.1" />
     <xacro:property name="wheel_length" value="0.05" />
-    <link name="base_foot_plane">
-    </link>
+    <link name="base_foot_plane" />
     <link name="base_link">
         <visual>
